Commit message: glb

File: public/kr1/urdf/kr1.urdf (robot description, URDF)
Before this commit: robot kr1, 7 links, 6 joints
Links:
- link Link1: geometry collision mesh filename=../meshes-glb/Link1.glb; visual mesh filename=../meshes-glb/Link1.glb
- link Link2: geometry collision mesh filename=../meshes-glb/Link2.glb; visual mesh filename=../meshes-glb/Link2.glb
- link Link3: geometry collision mesh filename=../meshes-glb/Link3.glb; visual mesh filename=../meshes-glb/Link3.glb
- link Link4: geometry collision mesh filename=../meshes-glb/Link4.glb; visual mesh filename=../meshes-glb/Link4.glb
- link Link5: geometry collision mesh filename=../meshes-glb/Link5.glb; visual mesh filename=../meshes-glb/Link5.glb
- link Link6: geometry collision mesh filename=../meshes-glb/Link6.glb; visual mesh filename=../meshes-glb/Link6.glb
- link base_link: geometry collision mesh filename=../meshes-glb/base_link.glb; visual mesh filename=../meshes-glb/base_link.glb
Joints:
- joint joint1: origin xyz=0 0 0.2452 rpy=0 0 3.1416 -> xyz=0 0 0.144  rpy=0 0 3.1416
- joint joint2: origin xyz=-0.14532 0.11129 0.2698 rpy=0 0 0 -> xyz=0 -0.06 0.097 rpy=0 0 0
- joint joint3: origin xyz=-0.55606 0.091003 0.53944 rpy=0 0 0 -> xyz=0 0.005 0.40 rpy=0 0 0
- joint joint4: origin xyz=-0.33086 -0.050063 0.10046 rpy=0 0 0 -> xyz=0 -0.005 0.33 rpy=0 0 0
- joint joint5: origin xyz=-0.55081 0.0018802 -0.13685 rpy=0 0 0 -> xyz=0 -0.071 0.05 rpy=0 0 0
- joint joint6: origin xyz=-0.12856 0.10531 0.0149 rpy=0 0 0 -> xyz=0 -0.05 0.057 rpy=0 0 0

Commit message: urdf glb

File: public/kr1/urdf/kr1.urdf (robot description, URDF)
Before this commit: robot kr1, 7 links, 6 joints
Joints:
- joint joint4: axis 0.97675 -0.14405 0.15878 -> 0 1 0
- joint joint5: axis 0.041475 0.85361 0.51927 -> 0 0 1
- joint joint6: axis 0.95243 -0.19082 0.23761 -> 0 1 0

Commit message: joint value basic

File: public/kr1/urdf/kr1.urdf (robot description, URDF)
Before this commit: robot kr1, 7 links, 6 joints
Joints:
- joint joint2: axis 0.1459 0.9893 0 -> 0 1 0
- joint joint3: axis 0.1459 0.9893 0 -> 0 1 0
